Commit message: implemented torsion suppression control based on vibration mode

File: robots/hydrus/robots/hex/hex_vibration_202004/robot.gazebo.xacro (robot description, xacro)
@@ -12,28 +12,28 @@
     <gazebo>
       <!-- joint torsional spring plugin -->
-      <plugin name="torsion1_r_torsional_spring" filename="libjoint_torsional_spring_plugin.so">
+      <plugin name="torsion1_torsional_spring" filename="libjoint_torsional_spring_plugin.so">
         <kx>5</kx>
         <set_point>0</set_point>
-        <joint>torsion1_r</joint>
+        <joint>torsion1</joint>
       </plugin>
-      <plugin name="torsion2_r_torsional_spring" filename="libjoint_torsional_spring_plugin.so">
+      <plugin name="torsion2_torsional_spring" filename="libjoint_torsional_spring_plugin.so">
         <kx>5</kx>
         <set_point>0</set_point>
-        <joint>torsion2_r</joint>
+        <joint>torsion2</joint>
       </plugin>
-      <plugin name="torsion3_r_torsional_spring" filename="libjoint_torsional_spring_plugin.so">
+      <plugin name="torsion3_torsional_spring" filename="libjoint_torsional_spring_plugin.so">
         <kx>5</kx>
         <set_point>0</set_point>
-        <joint>torsion3_r</joint>
+        <joint>torsion3</joint>
       </plugin>
-      <plugin name="torsion4_r_torsional_spring" filename="libjoint_torsional_spring_plugin.so">
+      <plugin name="torsion4_torsional_spring" filename="libjoint_torsional_spring_plugin.so">
         <kx>5</kx>
         <set_point>0</set_point>
-        <joint>torsion4_r</joint>
+        <joint>torsion4</joint>
       </plugin>
-      <plugin name="torsion5_r_torsional_spring" filename="libjoint_torsional_spring_plugin.so">
+      <plugin name="torsion5_torsional_spring" filename="libjoint_torsional_spring_plugin.so">
         <kx>5</kx>
         <set_point>0</set_point>
-        <joint>torsion5_r</joint>
+        <joint>torsion5</joint>
       </plugin>
     </gazebo>
@@ -41,5 +41,5 @@
       <plugin name="torsion_joint_state_publisher" filename="libgazebo_ros_joint_state_publisher.so">
         <robotNamespace>/$(arg robot_name)/link_torsion_groundtruth</robotNamespace>
-        <jointName>torsion1_r, torsion2_r, torsion3_r, torsion4_r, torsion5_r</jointName>
+        <jointName>torsion1, torsion2, torsion3, torsion4, torsion5</jointName>
         <!-- <robotNamespace>/$(arg robot_name)/link_torsion</robotNamespace> -->
         <!-- <jointName>torsion3_r</jointName> -->

File: robots/hydrus/robots/multi/multi_vibration_202007/robot.gazebo.xacro (robot description, xacro)
@@ -5,4 +5,5 @@
   <xacro:arg name="sim" default="false"/>
   <xacro:arg name="links" default="8"/>
+  <xacro:arg name="fix_rotor" default="0"/>
   <!-- robot urdf -->
   <xacro:include filename="$(find hydrus)/robots/multi/multi_vibration_202007/robot.urdf.xacro" />
@@ -14,8 +15,8 @@
     <gazebo>
     <xacro:macro name="loop_plugin_torsion" params="links_qty">
-      <plugin name="torsion${links_qty-1}_r_torsional_spring" filename="libjoint_torsional_spring_plugin.so">
+      <plugin name="torsion${links_qty-1}_torsional_spring" filename="libjoint_torsional_spring_plugin.so">
         <kx>10</kx>
         <set_point>0</set_point>
-        <joint>torsion${links_qty-1}_r</joint>
+        <joint>torsion${links_qty-1}</joint>
       </plugin>
       <xacro:if value="${links_qty-2}">
@@ -27,8 +28,8 @@
     <gazebo>
       <plugin name="torsion_joint_state_publisher" filename="libgazebo_ros_joint_state_publisher.so">
-        <robotNamespace>/$(arg robot_name)/link_torsion_groundtruth</robotNamespace>
-        <!-- <robotNamespace>/$(arg robot_name)/link_torsion</robotNamespace> -->
-        <!-- <jointName>torsion1_r, torsion2_r, torsion3_r, torsion4_r, torsion5_r</jointName> -->
-        <!-- <jointName>torsion1_r, torsion2_r, torsion3_r, torsion4_r, torsion5_r, torsion6_r, torsion7_r</jointName> -->
+        <!-- <robotNamespace>/$(arg robot_name)/link_torsion_groundtruth</robotNamespace> -->
+        <robotNamespace>/$(arg robot_name)/link_torsion</robotNamespace>
+        <jointName>torsion1, torsion2, torsion3, torsion4, torsion5</jointName>
+        <!-- <jointName>torsion1, torsion2, torsion3, torsion4, torsion5, torsion6, torsion7</jointName> -->
         <updateRate>30.0</updateRate>
         <alwaysOn>true</alwaysOn>

File: robots/hydrus/robots/multi/multi_vibration_202007/robot.urdf.xacro (robot description, xacro)
@@ -4,4 +4,5 @@
   <xacro:arg name="sim" default="false"/>
   <xacro:arg name="links" default="8"/>
+  <xacro:arg name="fix_rotor" default="0"/>
   <xacro:arg name="tilt_mode" default="1"/>
   <xacro:arg name="tilt_angle" default="20"/>
@@ -12,8 +13,8 @@
     <xacro:macro name="loop_link_sim" params="links_qty">
         <xacro:if value="${links_qty==$(arg links)}">
-          <xacro:hydrus_link links="$(arg links)" self="${links_qty}" rotor_direction="${int(pow(-1, links_qty))}" with_battery = "1"  vibrate = "0" tilt_mode="$(arg tilt_mode)" tilt_angle="$(arg tilt_angle)"/>
+          <xacro:hydrus_link links="$(arg links)" self="${links_qty}" rotor_direction="${int(pow(-1, links_qty))}" with_battery = "1"  vibrate = "0" tilt_mode="$(arg tilt_mode)" tilt_angle="$(arg tilt_angle)" fix_rotor="$(arg fix_rotor)"/>
         </xacro:if>
         <xacro:unless value="${links_qty==$(arg links)}">
-          <xacro:hydrus_link links="$(arg links)" self="${links_qty}" rotor_direction="${int(pow(-1, links_qty))}" with_battery = "1"  vibrate = "1" tilt_mode="$(arg tilt_mode)" tilt_angle="$(arg tilt_angle)"/>
+          <xacro:hydrus_link links="$(arg links)" self="${links_qty}" rotor_direction="${int(pow(-1, links_qty))}" with_battery = "1"  vibrate = "1" tilt_mode="$(arg tilt_mode)" tilt_angle="$(arg tilt_angle)" fix_rotor="$(arg fix_rotor)"/>
         </xacro:unless>
       <xacro:if value="${links_qty-1}">

File: robots/hydrus/urdf/link.urdf.xacro (robot description, xacro)
@@ -3,5 +3,5 @@
     xmlns:xacro="http://www.ros.org/wiki/xacro" name="hydrus_link" >
   <!-- D-H kai description(different from prof.nakamura) -->
-  <xacro:macro name="hydrus_link" params="links self rotor_direction with_leg:=1 with_battery:=1 old_version:=0 tilt_mode:=0 tilt_angle:=0 vibrate:=0">
+  <xacro:macro name="hydrus_link" params="links self rotor_direction with_leg:=1 with_battery:=1 old_version:=0 tilt_mode:=0 tilt_angle:=0 vibrate:=0 fix_rotor:=0">
     <xacro:if value="${old_version == 1}">
       <!-- link -->
@@ -143,5 +143,11 @@
     <xacro:damping_factor link ="link${self}"/>
     <!-- rotor -->
-    <joint name="rotor${self}" type="continuous">
+    <xacro:if value="${fix_rotor == 1}">
+      <xacro:property name="rotor_joint_type" value="fixed"/>
+    </xacro:if>
+    <xacro:unless value="${fix_rotor == 1}">
+      <xacro:property name="rotor_joint_type" value="continuous"/>
+    </xacro:unless>
+    <joint name="rotor${self}" type="${rotor_joint_type}">
       <limit effort="100.0" lower="${min_force}" upper="${max_force}" velocity="0.5"/>
       <parent link="link${self}"/>
@@ -233,5 +239,5 @@
     <xacro:unless value="${self == links}">
       <xacro:if value="${vibrate == 1}">
-        <link name="torsion_dummy${self}_r">
+        <link name="torsion_dummy${self}">
           <inertial>
             <origin xyz="0 0 0" rpy="0 0 0"/>
@@ -243,8 +249,8 @@
           </inertial>
         </link>
-        <joint name="torsion${self}_r" type="revolute">
+        <joint name="torsion${self}" type="revolute">
           <limit effort="10000.0" lower="${-pi/6}" upper="${pi/6}" velocity="1"/>
           <parent link="link${self}"/>
-          <child link="torsion_dummy${self}_r"/>
+          <child link="torsion_dummy${self}"/>
           <origin rpy="0 0 0" xyz="${link_length} 0 0"/>
           <axis xyz="1 0 0"/>
@@ -278,5 +284,5 @@
         </xacro:unless>
         <xacro:if value="${vibrate == 1}">
-          <parent link="torsion_dummy${self}_r"/>
+          <parent link="torsion_dummy${self}"/>
           <child link="link${self+1}"/>
           <!-- <child link="torsion_dummy${self}_l"/> -->
