Commit message: modified simulation parameters according to experiments

File: robots/hydrus/robots/hex/hex_vibration_mode_202007/robot.gazebo.xacro (robot description, xacro)
@@ -14,25 +14,25 @@
       <!-- joint torsional spring plugin -->
       <plugin name="torsion1_torsional_spring" filename="libjoint_torsional_spring_plugin.so">
-        <kx>10</kx>
+        <kx>60</kx>
         <set_point>0</set_point>
         <joint>torsion1</joint>
       </plugin>
       <plugin name="torsion2_torsional_spring" filename="libjoint_torsional_spring_plugin.so">
-        <kx>10</kx>
+        <kx>60</kx>
         <set_point>0</set_point>
         <joint>torsion2</joint>
       </plugin>
       <plugin name="torsion3_torsional_spring" filename="libjoint_torsional_spring_plugin.so">
-        <kx>10</kx>
+        <kx>60</kx>
         <set_point>0</set_point>
         <joint>torsion3</joint>
       </plugin>
       <plugin name="torsion4_torsional_spring" filename="libjoint_torsional_spring_plugin.so">
-        <kx>10</kx>
+        <kx>60</kx>
         <set_point>0</set_point>
         <joint>torsion4</joint>
       </plugin>
       <plugin name="torsion5_torsional_spring" filename="libjoint_torsional_spring_plugin.so">
-        <kx>10</kx>
+        <kx>60</kx>
         <set_point>0</set_point>
         <joint>torsion5</joint>
@@ -42,8 +42,7 @@
       <plugin name="torsion_joint_state_publisher" filename="libgazebo_ros_joint_state_publisher.so">
         <robotNamespace>/$(arg robot_name)/link_torsion_groundtruth</robotNamespace>
+        <!-- <robotNamespace>/$(arg robot_name)/link_torsion</robotNamespace> -->
         <jointName>torsion1, torsion2, torsion3, torsion4, torsion5</jointName>
-        <!-- <robotNamespace>/$(arg robot_name)/link_torsion</robotNamespace> -->
-        <!-- <jointName>torsion3_r</jointName> -->
-        <updateRate>50.0</updateRate>
+        <updateRate>60.0</updateRate>
         <alwaysOn>true</alwaysOn>
       </plugin>
@@ -62,5 +61,6 @@
         <bodyName>neuron1_imu</bodyName>
         <updateRateHZ>200.0</updateRateHZ>
-        <gaussianNoise>0.001</gaussianNoise>
+        <!-- <gaussianNoise>0.001</gaussianNoise> -->
+        <gaussianNoise>0</gaussianNoise>
         <xyzOffset>0 0 0</xyzOffset>
         <rpyOffset>0 0 0</rpyOffset>
@@ -81,8 +81,84 @@
         <bodyName>main_imu</bodyName>
         <updateRateHZ>200.0</updateRateHZ>
-        <gaussianNoise>0.001</gaussianNoise>
+        <gaussianNoise>0</gaussianNoise>
         <xyzOffset>0 0 0</xyzOffset>
         <rpyOffset>0 0 0</rpyOffset>
         <frameName>fc</frameName>
+      </plugin>
+      <pose>0 0 0 0 0 0</pose>
+    </sensor>
+  </gazebo>
+  <gazebo reference="neuron2_imu">
+    <gravity>true</gravity>
+    <sensor name="neuron2_imu" type="imu">
+      <always_on>true</always_on>
+      <update_rate>100</update_rate>
+      <visualize>true</visualize>
+      <topic>__default_topic__</topic>
+      <plugin filename="libgazebo_ros_imu_sensor.so" name="imu_plugin">
+        <topicName>/$(arg robot_name)/neuron2_imu</topicName>
+        <bodyName>neuron2_imu</bodyName>
+        <updateRateHZ>200.0</updateRateHZ>
+        <gaussianNoise>0</gaussianNoise>
+        <xyzOffset>0 0 0</xyzOffset>
+        <rpyOffset>0 0 0</rpyOffset>
+        <frameName>neuron2_imu</frameName>
+      </plugin>
+      <pose>0 0 0 0 0 0</pose>
+    </sensor>
+  </gazebo>
+  <gazebo reference="neuron3_imu">
+    <gravity>true</gravity>
+    <sensor name="neuron3_imu" type="imu">
+      <always_on>true</always_on>
+      <update_rate>100</update_rate>
+      <visualize>true</visualize>
+      <topic>__default_topic__</topic>
+      <plugin filename="libgazebo_ros_imu_sensor.so" name="imu_plugin">
+        <topicName>/$(arg robot_name)/neuron3_imu</topicName>
+        <bodyName>neuron3_imu</bodyName>
+        <updateRateHZ>200.0</updateRateHZ>
+        <gaussianNoise>0</gaussianNoise>
+        <xyzOffset>0 0 0</xyzOffset>
+        <rpyOffset>0 0 0</rpyOffset>
+        <frameName>neuron3_imu</frameName>
+      </plugin>
+      <pose>0 0 0 0 0 0</pose>
+    </sensor>
+  </gazebo>
+  <gazebo reference="neuron4_imu">
+    <gravity>true</gravity>
+    <sensor name="neuron4_imu" type="imu">
+      <always_on>true</always_on>
+      <update_rate>100</update_rate>
+      <visualize>true</visualize>
+      <topic>__default_topic__</topic>
+      <plugin filename="libgazebo_ros_imu_sensor.so" name="imu_plugin">
+        <topicName>/$(arg robot_name)/neuron4_imu</topicName>
+        <bodyName>neuron4_imu</bodyName>
+        <updateRateHZ>200.0</updateRateHZ>
+        <gaussianNoise>0</gaussianNoise>
+        <xyzOffset>0 0 0</xyzOffset>
+        <rpyOffset>0 0 0</rpyOffset>
+        <frameName>neuron4_imu</frameName>
+      </plugin>
+      <pose>0 0 0 0 0 0</pose>
+    </sensor>
+  </gazebo>
+  <gazebo reference="neuron5_imu">
+    <gravity>true</gravity>
+    <sensor name="neuron5_imu" type="imu">
+      <always_on>true</always_on>
+      <update_rate>100</update_rate>
+      <visualize>true</visualize>
+      <topic>__default_topic__</topic>
+      <plugin filename="libgazebo_ros_imu_sensor.so" name="imu_plugin">
+        <topicName>/$(arg robot_name)/neuron5_imu</topicName>
+        <bodyName>neuron5_imu</bodyName>
+        <updateRateHZ>200.0</updateRateHZ>
+        <gaussianNoise>0</gaussianNoise>
+        <xyzOffset>0 0 0</xyzOffset>
+        <rpyOffset>0 0 0</rpyOffset>
+        <frameName>neuron5_imu</frameName>
       </plugin>
       <pose>0 0 0 0 0 0</pose>
@@ -100,5 +176,5 @@
         <bodyName>neuron6_imu</bodyName>
         <updateRateHZ>200.0</updateRateHZ>
-        <gaussianNoise>0.001</gaussianNoise>
+        <gaussianNoise>0</gaussianNoise>
         <xyzOffset>0 0 0</xyzOffset>
         <rpyOffset>0 0 0</rpyOffset>
@@ -113,8 +189,44 @@
     <!-- TODO neuron?_imu does not work as bodyName why? -->
     <plugin filename="libgazebo_ros_p3d.so" name="neuron1_groundtruth">
-      <bodyName>thrust1</bodyName>
+      <bodyName>link1</bodyName>
       <topicName>/$(arg robot_name)/neuron1_groundtruth</topicName>
-      <updateRate>50</updateRate>
-      <gaussianNoise>0.005</gaussianNoise>
+      <updateRate>100</updateRate>
+      <gaussianNoise>0.001</gaussianNoise>
+      <xyzOffset>0 0 0</xyzOffset>
+      <rpyOffset>0 0 0</rpyOffset>
+      <frameName>world</frameName>
+    </plugin>
+    <plugin filename="libgazebo_ros_p3d.so" name="neuron2_groundtruth">
+      <bodyName>link2</bodyName>
+      <topicName>/$(arg robot_name)/neuron2_groundtruth</topicName>
+      <updateRate>100</updateRate>
+      <gaussianNoise>0.001</gaussianNoise>
+      <xyzOffset>0 0 0</xyzOffset>
+      <rpyOffset>0 0 0</rpyOffset>
+      <frameName>world</frameName>
+    </plugin>
+    <plugin filename="libgazebo_ros_p3d.so" name="neuron3_groundtruth">
+      <bodyName>link3</bodyName>
+      <topicName>/$(arg robot_name)/neuron3_groundtruth</topicName>
+      <updateRate>100</updateRate>
+      <gaussianNoise>0.001</gaussianNoise>
+      <xyzOffset>0 0 0</xyzOffset>
+      <rpyOffset>0 0 0</rpyOffset>
+      <frameName>world</frameName>
+    </plugin>
+    <plugin filename="libgazebo_ros_p3d.so" name="neuron4_groundtruth">
+      <bodyName>link4</bodyName>
+      <topicName>/$(arg robot_name)/neuron4_groundtruth</topicName>
+      <updateRate>100</updateRate>
+      <gaussianNoise>0.001</gaussianNoise>
+      <xyzOffset>0 0 0</xyzOffset>
+      <rpyOffset>0 0 0</rpyOffset>
+      <frameName>world</frameName>
+    </plugin>
+    <plugin filename="libgazebo_ros_p3d.so" name="neuron5_groundtruth">
+      <bodyName>link5</bodyName>
+      <topicName>/$(arg robot_name)/neuron5_groundtruth</topicName>
+      <updateRate>100</updateRate>
+      <gaussianNoise>0.001</gaussianNoise>
       <xyzOffset>0 0 0</xyzOffset>
       <rpyOffset>0 0 0</rpyOffset>
@@ -122,8 +234,8 @@
     </plugin>
     <plugin filename="libgazebo_ros_p3d.so" name="neuron6_groundtruth">
-      <bodyName>thrust6</bodyName>
+      <bodyName>link6</bodyName>
       <topicName>/$(arg robot_name)/neuron6_groundtruth</topicName>
-      <updateRate>50</updateRate>
-      <gaussianNoise>0.005</gaussianNoise>
+      <updateRate>100</updateRate>
+      <gaussianNoise>0.001</gaussianNoise>
       <xyzOffset>0 0 0</xyzOffset>
       <rpyOffset>0 0 0</rpyOffset>

File: robots/hydrus/robots/hex/hex_vibration_mode_202007/robot.urdf.xacro (robot description, xacro)
@@ -131,4 +131,48 @@
     </inertial>
   </xacro:extra_module>
+  <xacro:extra_module name = "neuron2_imu" parent = "link2">
+    <origin xyz="${0.03} 0 ${0.02}" rpy="0 0 0"/>
+    <inertial>
+      <mass value = "0.00001" />
+      <origin xyz="0 0 0" rpy="0 0 0"/>
+      <inertia
+          ixx="0.000001" ixy="0.0" ixz="0.0"
+          iyy="0.000001" iyz="0.0"
+          izz="0.000002"/>
+    </inertial>
+  </xacro:extra_module>
+  <xacro:extra_module name = "neuron3_imu" parent = "link3">
+    <origin xyz="${0.03} 0 ${0.02}" rpy="0 0 0"/>
+    <inertial>
+      <mass value = "0.00001" />
+      <origin xyz="0 0 0" rpy="0 0 0"/>
+      <inertia
+          ixx="0.000001" ixy="0.0" ixz="0.0"
+          iyy="0.000001" iyz="0.0"
+          izz="0.000002"/>
+    </inertial>
+  </xacro:extra_module>
+  <xacro:extra_module name = "neuron4_imu" parent = "link4">
+    <origin xyz="${0.03} 0 ${0.02}" rpy="0 0 0"/>
+    <inertial>
+      <mass value = "0.00001" />
+      <origin xyz="0 0 0" rpy="0 0 0"/>
+      <inertia
+          ixx="0.000001" ixy="0.0" ixz="0.0"
+          iyy="0.000001" iyz="0.0"
+          izz="0.000002"/>
+    </inertial>
+  </xacro:extra_module>
+  <xacro:extra_module name = "neuron5_imu" parent = "link5">
+    <origin xyz="${0.03} 0 ${0.02}" rpy="0 0 0"/>
+    <inertial>
+      <mass value = "0.00001" />
+      <origin xyz="0 0 0" rpy="0 0 0"/>
+      <inertia
+          ixx="0.000001" ixy="0.0" ixz="0.0"
+          iyy="0.000001" iyz="0.0"
+          izz="0.000002"/>
+    </inertial>
+  </xacro:extra_module>
   <xacro:extra_module name = "neuron6_imu" parent = "link6">
     <origin xyz="${link_length - 0.03} 0 ${0.02}" rpy="0 0 0"/>

File: robots/hydrus/robots/multi/multi_vibration_202007/robot.gazebo.xacro (robot description, xacro)
@@ -30,5 +30,5 @@
         <robotNamespace>/$(arg robot_name)/link_torsion_groundtruth</robotNamespace>
         <!-- <robotNamespace>/$(arg robot_name)/link_torsion</robotNamespace> -->
-        <jointName>torsion1, torsion2, torsion3, torsion4, torsion5</jointName>
+        <!-- <jointName>torsion1, torsion2, torsion3, torsion4, torsion5</jointName> -->
         <!-- <jointName>torsion1, torsion2, torsion3, torsion4, torsion5, torsion6, torsion7</jointName> -->
         <updateRate>30.0</updateRate>

File: robots/hydrus/urdf/link.urdf.xacro (robot description, xacro)
@@ -250,10 +250,10 @@
         </link>
         <joint name="torsion${self}" type="revolute">
-          <limit effort="10000.0" lower="${-pi/6}" upper="${pi/6}" velocity="1"/>
+          <limit effort="10000.0" lower="${-pi/4}" upper="${pi/4}" velocity="1"/>
           <parent link="link${self}"/>
           <child link="torsion_dummy${self}"/>
           <origin rpy="0 0 0" xyz="${link_length} 0 0"/>
           <axis xyz="1 0 0"/>
-          <dynamics damping="0.9" friction="0.05"/>
+          <dynamics damping="0.7" friction="0.00"/>
         </joint>
         <!-- <link name="torsion_dummy${self}_l"> -->

Commit message: added torsion estimator

File: robots/hydrus/robots/hex/hex_vibration_mode_202007/robot.gazebo.xacro (robot description, xacro)
@@ -54,5 +54,5 @@
     <sensor name="neuron1_imu" type="imu">
       <always_on>true</always_on>
-      <update_rate>100</update_rate>
+      <update_rate>60</update_rate>
       <visualize>true</visualize>
       <topic>__default_topic__</topic>
@@ -60,5 +60,5 @@
         <topicName>/$(arg robot_name)/neuron1_imu</topicName>
         <bodyName>neuron1_imu</bodyName>
-        <updateRateHZ>200.0</updateRateHZ>
+        <updateRateHZ>60.0</updateRateHZ>
         <!-- <gaussianNoise>0.001</gaussianNoise> -->
         <gaussianNoise>0</gaussianNoise>
@@ -74,5 +74,5 @@
     <sensor name="main_imu" type="imu">
       <always_on>true</always_on>
-      <update_rate>100</update_rate>
+      <update_rate>60</update_rate>
       <visualize>true</visualize>
       <topic>__default_topic__</topic>
@@ -80,5 +80,5 @@
         <topicName>/$(arg robot_name)/main_imu</topicName>
         <bodyName>main_imu</bodyName>
-        <updateRateHZ>200.0</updateRateHZ>
+        <updateRateHZ>60.0</updateRateHZ>
         <gaussianNoise>0</gaussianNoise>
         <xyzOffset>0 0 0</xyzOffset>
@@ -93,5 +93,5 @@
     <sensor name="neuron2_imu" type="imu">
       <always_on>true</always_on>
-      <update_rate>100</update_rate>
+      <update_rate>60</update_rate>
       <visualize>true</visualize>
       <topic>__default_topic__</topic>
@@ -99,5 +99,5 @@
         <topicName>/$(arg robot_name)/neuron2_imu</topicName>
         <bodyName>neuron2_imu</bodyName>
-        <updateRateHZ>200.0</updateRateHZ>
+        <updateRateHZ>60.0</updateRateHZ>
         <gaussianNoise>0</gaussianNoise>
         <xyzOffset>0 0 0</xyzOffset>
@@ -112,5 +112,5 @@
     <sensor name="neuron3_imu" type="imu">
       <always_on>true</always_on>
-      <update_rate>100</update_rate>
+      <update_rate>60</update_rate>
       <visualize>true</visualize>
       <topic>__default_topic__</topic>
@@ -118,5 +118,5 @@
         <topicName>/$(arg robot_name)/neuron3_imu</topicName>
         <bodyName>neuron3_imu</bodyName>
-        <updateRateHZ>200.0</updateRateHZ>
+        <updateRateHZ>60.0</updateRateHZ>
         <gaussianNoise>0</gaussianNoise>
         <xyzOffset>0 0 0</xyzOffset>
@@ -131,5 +131,5 @@
     <sensor name="neuron4_imu" type="imu">
       <always_on>true</always_on>
-      <update_rate>100</update_rate>
+      <update_rate>60</update_rate>
       <visualize>true</visualize>
       <topic>__default_topic__</topic>
@@ -137,5 +137,5 @@
         <topicName>/$(arg robot_name)/neuron4_imu</topicName>
         <bodyName>neuron4_imu</bodyName>
-        <updateRateHZ>200.0</updateRateHZ>
+        <updateRateHZ>60.0</updateRateHZ>
         <gaussianNoise>0</gaussianNoise>
         <xyzOffset>0 0 0</xyzOffset>
@@ -150,5 +150,5 @@
     <sensor name="neuron5_imu" type="imu">
       <always_on>true</always_on>
-      <update_rate>100</update_rate>
+      <update_rate>60</update_rate>
       <visualize>true</visualize>
       <topic>__default_topic__</topic>
@@ -156,5 +156,5 @@
         <topicName>/$(arg robot_name)/neuron5_imu</topicName>
         <bodyName>neuron5_imu</bodyName>
-        <updateRateHZ>200.0</updateRateHZ>
+        <updateRateHZ>60.0</updateRateHZ>
         <gaussianNoise>0</gaussianNoise>
         <xyzOffset>0 0 0</xyzOffset>
@@ -169,5 +169,5 @@
     <sensor name="neuron6_imu" type="imu">
       <always_on>true</always_on>
-      <update_rate>100</update_rate>
+      <update_rate>60</update_rate>
       <visualize>true</visualize>
       <topic>__default_topic__</topic>
@@ -175,5 +175,5 @@
         <topicName>/$(arg robot_name)/neuron6_imu</topicName>
         <bodyName>neuron6_imu</bodyName>
-        <updateRateHZ>200.0</updateRateHZ>
+        <updateRateHZ>60.0</updateRateHZ>
         <gaussianNoise>0</gaussianNoise>
         <xyzOffset>0 0 0</xyzOffset>
@@ -190,5 +190,5 @@
     <plugin filename="libgazebo_ros_p3d.so" name="neuron1_groundtruth">
       <bodyName>link1</bodyName>
-      <topicName>/$(arg robot_name)/neuron1_groundtruth</topicName>
+      <topicName>/$(arg robot_name)/mocap/link1/pose</topicName>
       <updateRate>100</updateRate>
       <gaussianNoise>0.001</gaussianNoise>
@@ -199,5 +199,5 @@
     <plugin filename="libgazebo_ros_p3d.so" name="neuron2_groundtruth">
       <bodyName>link2</bodyName>
-      <topicName>/$(arg robot_name)/neuron2_groundtruth</topicName>
+      <topicName>/$(arg robot_name)/mocap/link2/pose</topicName>
       <updateRate>100</updateRate>
       <gaussianNoise>0.001</gaussianNoise>
@@ -208,5 +208,5 @@
     <plugin filename="libgazebo_ros_p3d.so" name="neuron3_groundtruth">
       <bodyName>link3</bodyName>
-      <topicName>/$(arg robot_name)/neuron3_groundtruth</topicName>
+      <topicName>/$(arg robot_name)/mocap/link3/pose</topicName>
       <updateRate>100</updateRate>
       <gaussianNoise>0.001</gaussianNoise>
@@ -217,5 +217,5 @@
     <plugin filename="libgazebo_ros_p3d.so" name="neuron4_groundtruth">
       <bodyName>link4</bodyName>
-      <topicName>/$(arg robot_name)/neuron4_groundtruth</topicName>
+      <topicName>/$(arg robot_name)/mocap/link4/pose</topicName>
       <updateRate>100</updateRate>
       <gaussianNoise>0.001</gaussianNoise>
@@ -226,5 +226,5 @@
     <plugin filename="libgazebo_ros_p3d.so" name="neuron5_groundtruth">
       <bodyName>link5</bodyName>
-      <topicName>/$(arg robot_name)/neuron5_groundtruth</topicName>
+      <topicName>/$(arg robot_name)/mocap/link5/pose</topicName>
       <updateRate>100</updateRate>
       <gaussianNoise>0.001</gaussianNoise>
@@ -235,5 +235,5 @@
     <plugin filename="libgazebo_ros_p3d.so" name="neuron6_groundtruth">
       <bodyName>link6</bodyName>
-      <topicName>/$(arg robot_name)/neuron6_groundtruth</topicName>
+      <topicName>/$(arg robot_name)/mocap/link6/pose</topicName>
       <updateRate>100</updateRate>
       <gaussianNoise>0.001</gaussianNoise>

File: robots/hydrus/robots/hex/hex_vibration_mode_202007/robot.urdf.xacro (robot description, xacro)
@@ -6,7 +6,13 @@
   <xacro:arg name="tilt_mode" default="1"/>
   <xacro:arg name="tilt_angle" default="20"/>
+  <xacro:arg name="root_on_fc" default="false"/>
   <!-- basic kinematics model -->
   <xacro:include filename="$(find hydrus)/urdf/common.xacro" />
-  <xacro:include filename="$(find hydrus)/urdf/link.urdf.xacro" />
+  <xacro:unless value="$(arg root_on_fc)">
+    <xacro:include filename="$(find hydrus)/urdf/link.urdf.xacro" />
+  </xacro:unless>
+  <xacro:if value="$(arg root_on_fc)">
+    <xacro:include filename="$(find hydrus)/urdf/link_root_on_fc.urdf.xacro" />
+  </xacro:if>
   <xacro:if value="$(arg sim)">
     <xacro:hydrus_link links="6" self="1" rotor_direction="-1" with_battery = "1"  vibrate = "1" tilt_mode="$(arg tilt_mode)" tilt_angle="$(arg tilt_angle)" fix_rotor="$(arg fix_rotor)"/>
@@ -176,5 +182,6 @@
   </xacro:extra_module>
   <xacro:extra_module name = "neuron6_imu" parent = "link6">
-    <origin xyz="${link_length - 0.03} 0 ${0.02}" rpy="0 0 0"/>
+    <origin xyz="${0.03} 0 ${0.02}" rpy="0 0 0"/>
+    <!-- <origin xyz="${link_length - 0.03} 0 ${0.02}" rpy="0 0 0"/> -->
     <inertial>
       <mass value = "0.00001" />
