Commit message: refactored torsion control

File: robots/hydrus/robots/hex/hex_vibration_mode_202007/robot.urdf.xacro (robot description, xacro)
@@ -6,13 +6,7 @@
   <xacro:arg name="tilt_mode" default="1"/>
   <xacro:arg name="tilt_angle" default="20"/>
-  <xacro:arg name="root_on_fc" default="false"/>
   <!-- basic kinematics model -->
   <xacro:include filename="$(find hydrus)/urdf/common.xacro" />
-  <xacro:unless value="$(arg root_on_fc)">
-    <xacro:include filename="$(find hydrus)/urdf/link.urdf.xacro" />
-  </xacro:unless>
-  <xacro:if value="$(arg root_on_fc)">
-    <xacro:include filename="$(find hydrus)/urdf/link_root_on_fc.urdf.xacro" />
-  </xacro:if>
+  <xacro:include filename="$(find hydrus)/urdf/link.urdf.xacro" />
   <xacro:if value="$(arg sim)">
     <xacro:hydrus_link links="6" self="1" rotor_direction="-1" with_battery = "1"  vibrate = "1" tilt_mode="$(arg tilt_mode)" tilt_angle="$(arg tilt_angle)" fix_rotor="$(arg fix_rotor)"/>

File: robots/hydrus/robots/multi/multi_vibration_202007/robot.urdf.xacro (robot description, xacro)
@@ -5,15 +5,9 @@
   <xacro:arg name="links" default="8"/>
   <xacro:arg name="fix_rotor" default="0"/>
-  <xacro:arg name="root_on_fc" default="0"/>
   <xacro:arg name="tilt_mode" default="1"/>
   <xacro:arg name="tilt_angle" default="20"/>
   <!-- basic kinematics model -->
   <xacro:include filename="$(find hydrus)/urdf/common.xacro" />
-  <xacro:unless value="${$(arg root_on_fc)==1}">
-    <xacro:include filename="$(find hydrus)/urdf/link.urdf.xacro" />
-  </xacro:unless>
-  <xacro:if value="${$(arg root_on_fc)==1}">
-    <xacro:include filename="$(find hydrus)/urdf/link_root_on_fc.urdf.xacro" />
-  </xacro:if>
+  <xacro:include filename="$(find hydrus)/urdf/link.urdf.xacro" />
   <xacro:if value="$(arg sim)">
     <xacro:macro name="loop_link_sim" params="links_qty">

File: robots/hydrus/robots/oct/oct_vibration_shift_202011/robot.gazebo.xacro (robot description, xacro)
@@ -6,5 +6,5 @@
   <xacro:arg name="fix_rotor" default="0"/>
   <!-- robot urdf -->
-  <xacro:include filename="$(find hydrus)/robots/oct/oct_vibration_mode_202010/robot.urdf.xacro" />
+  <xacro:include filename="$(find hydrus)/robots/oct/oct_vibration_shift_202011/robot.urdf.xacro" />
   <!-- gazebo plugin for default controller and sensors -->
   <xacro:include filename="$(find aerial_robot_simulation)/xacro/spinal.gazebo.xacro" />

File: robots/hydrus/urdf/link.urdf.xacro (robot description, xacro)
@@ -10,4 +10,5 @@
     <xacro:property name="link_inertial_pos" value="0.5"/>
   </xacro:unless>
+  <xacro:property name="link_half_mass_for_dummy" value="0.3"/>
     <xacro:if value="${old_version == 1}">
       <!-- link -->
@@ -17,5 +18,5 @@
           <inertial>
             <origin xyz="${link_length* link_inertial_pos + 0.055120} 0.0 0.011580" rpy="0 0 0"/>
-            <mass value="${0.566650-0.3*vibrate}"/>
+            <mass value="${0.566650-link_half_mass_for_dummy*vibrate}"/>
             <inertia
                 ixx="0.001804" iyy="0.017972" izz="0.019248"
@@ -29,5 +30,5 @@
             <inertial>
               <origin xyz="${link_length * link_inertial_pos + -0.013450} 0.0 0.012830" rpy="0 0 0"/>
-              <mass value="${0.495530-0.3*vibrate}"/>
+              <mass value="${0.495530-link_half_mass_for_dummy*vibrate}"/>
               <inertia
                   ixx="0.001758" iyy="0.013619" izz="0.014910"
@@ -40,5 +41,5 @@
             <inertial>
               <origin xyz="${link_length * link_inertial_pos + 0.038190} 0.0 0.010950" rpy="0 0 0"/>
-              <mass value="${0.597720-0.3*vibrate}"/>
+              <mass value="${0.597720-link_half_mass_for_dummy*vibrate}"/>
               <inertia
                   ixx="0.001828" iyy="0.021127" izz="0.022388"
@@ -67,5 +68,5 @@
             <inertial>
               <origin xyz="${link_length* link_inertial_pos + 0.057} 0.0 0.018" rpy="0 0 0"/>
-              <mass value="${0.58712-0.3*vibrate}"/>
+              <mass value="${0.58712-link_half_mass_for_dummy*vibrate}"/>
               <inertia
                   ixx="0.00179" iyy="0.01605" izz="0.01714"
@@ -81,5 +82,5 @@
               <inertial>
                 <origin xyz="${link_length* link_inertial_pos - 0.0576} 0.0 0.0258" rpy="0 0 0"/>
-                <mass value="${0.616-0.3*vibrate}"/>
+                <mass value="${0.616-link_half_mass_for_dummy*vibrate}"/>
                 <inertia
                     ixx="0.002" iyy="0.0161" izz="0.016992"
@@ -90,5 +91,5 @@
               <inertial>
                 <origin xyz="${link_length * link_inertial_pos -0.058} 0.0 0.0188" rpy="0 0 0"/>
-                <mass value="${0.590-0.3*vibrate}"/> <!-- +DCDC -->
+                <mass value="${0.590-link_half_mass_for_dummy*vibrate}"/> <!-- +DCDC -->
                 <inertia
                     ixx="0.00179" iyy="0.01581" izz="0.01692"
@@ -104,5 +105,5 @@
                 <inertial>
                   <origin xyz="${link_length* link_inertial_pos - 0.0005} 0.0 0.0204" rpy="0 0 0"/>
-                  <mass value="${0.58312-0.3*vibrate}"/>
+                  <mass value="${0.58312-link_half_mass_for_dummy*vibrate}"/>
                   <inertia
                       ixx="0.002" iyy="0.01752" izz="0.018447"
@@ -113,5 +114,5 @@
                 <inertial>
                   <origin xyz="${link_length * link_inertial_pos} 0.0 0.01287" rpy="0 0 0"/>
-                  <mass value="${0.55744-0.3*vibrate}"/>
+                  <mass value="${0.55744-link_half_mass_for_dummy*vibrate}"/>
                   <inertia
                       ixx="0.00171" iyy="0.01727" izz="0.01844"
@@ -126,5 +127,5 @@
                 <inertial>
                   <origin xyz="${link_length* link_inertial_pos - 0.03} 0.0 0.025" rpy="0 0 0"/>
-                  <mass value="${0.66183-0.3*vibrate}"/>
+                  <mass value="${0.66183-link_half_mass_for_dummy*vibrate}"/>
                   <inertia
                       ixx="0.002" iyy="0.021851" izz="0.022718"
@@ -135,5 +136,5 @@
                 <inertial>
                   <origin xyz="${link_length * link_inertial_pos - 0.0317} 0.0 0.01836" rpy="0 0 0"/>
-                  <mass value="${0.63453-0.3*vibrate}"/>
+                  <mass value="${0.63453-link_half_mass_for_dummy*vibrate}"/>
                   <inertia
                       ixx="0.00182" iyy="0.02232" izz="0.02254"
@@ -248,5 +249,5 @@
           <inertial>
             <origin xyz="${link_length*0.25} 0 0.012" rpy="0 0 0"/>
-            <mass value="0.3"/>
+            <mass value="${link_half_mass_for_dummy}"/>
             <inertia
                 ixx="0.001828" iyy="0.021127" izz="0.022388"
