Commit message: implemented gain shift using null space for hydrus vibration suppression

File: robots/hydrus/robots/oct/oct_vibration_mode_202010/robot.gazebo.xacro (robot description, xacro)
@@ -5,4 +5,5 @@
   <xacro:arg name="sim" default="false"/>
   <xacro:arg name="fix_rotor" default="0"/>
+  <xacro:arg name="root_on_fc" default="false"/>
   <!-- robot urdf -->
   <xacro:include filename="$(find hydrus)/robots/oct/oct_vibration_mode_202010/robot.urdf.xacro" />

File: robots/hydrus/urdf/common.xacro (robot description, xacro)
@@ -130,5 +130,5 @@
   <xacro:macro name="damping_factor" params="link">
     <gazebo reference="${link}">
-      <dampingFactor>0.00</dampingFactor>
+      <dampingFactor>0.001</dampingFactor>
     </gazebo>
   </xacro:macro>

File: robots/hydrus/urdf/link.urdf.xacro (robot description, xacro)
@@ -4,4 +4,10 @@
   <!-- D-H kai description(different from prof.nakamura) -->
   <xacro:macro name="hydrus_link" params="links self rotor_direction with_leg:=1 with_battery:=1 old_version:=0 tilt_mode:=0 tilt_angle:=0 vibrate:=0 fix_rotor:=0">
+  <xacro:if value="${vibrate==1}">
+    <xacro:property name="link_inertial_pos" value="0.25"/>
+  </xacro:if>
+  <xacro:unless value="${vibrate==1}">
+    <xacro:property name="link_inertial_pos" value="0.5"/>
+  </xacro:unless>
     <xacro:if value="${old_version == 1}">
       <!-- link -->
@@ -10,6 +16,6 @@
         <xacro:if value="${self == 1}">
           <inertial>
-            <origin xyz="${link_length* 0.5 + 0.055120} 0.0 0.011580" rpy="0 0 0"/>
-            <mass value="0.566650"/>
+            <origin xyz="${link_length* link_inertial_pos + 0.055120} 0.0 0.011580" rpy="0 0 0"/>
+            <mass value="${0.566650-0.3*vibrate}"/>
             <inertia
                 ixx="0.001804" iyy="0.017972" izz="0.019248"
@@ -22,6 +28,6 @@
           <xacro:if value="${self == links}">
             <inertial>
-              <origin xyz="${link_length * 0.5 + -0.013450} 0.0 0.012830" rpy="0 0 0"/>
-              <mass value="0.495530"/>
+              <origin xyz="${link_length * link_inertial_pos + -0.013450} 0.0 0.012830" rpy="0 0 0"/>
+              <mass value="${0.495530-0.3*vibrate}"/>
               <inertia
                   ixx="0.001758" iyy="0.013619" izz="0.014910"
@@ -33,6 +39,6 @@
             <!-- general -->
             <inertial>
-              <origin xyz="${link_length * 0.5 + 0.038190} 0.0 0.010950" rpy="0 0 0"/>
-              <mass value="0.597720"/>
+              <origin xyz="${link_length * link_inertial_pos + 0.038190} 0.0 0.010950" rpy="0 0 0"/>
+              <mass value="${0.597720-0.3*vibrate}"/>
               <inertia
                   ixx="0.001828" iyy="0.021127" izz="0.022388"
@@ -51,6 +57,6 @@
           <xacro:if value="${tilt_mode == 1}">
             <inertial>
-              <origin xyz="${link_length* 0.5 + 0.056} 0.0 0.02577" rpy="0 0 0"/>
-              <mass value="0.61442"/>
+              <origin xyz="${link_length* link_inertial_pos + 0.056} 0.0 0.02577" rpy="0 0 0"/>
+              <mass value="${0.61442-0.3*vibrate}"/>
               <inertia
                   ixx="0.002" iyy="0.01634" izz="0.01723"
@@ -60,6 +66,6 @@
           <xacro:unless value="${tilt_mode == 1}">
             <inertial>
-              <origin xyz="${link_length* 0.5 + 0.057} 0.0 0.018" rpy="0 0 0"/>
-              <mass value="0.58712"/>
+              <origin xyz="${link_length* link_inertial_pos + 0.057} 0.0 0.018" rpy="0 0 0"/>
+              <mass value="${0.58712-0.3*vibrate}"/>
               <inertia
                   ixx="0.00179" iyy="0.01605" izz="0.01714"
@@ -74,6 +80,6 @@
             <xacro:if value="${tilt_mode == 1}">
               <inertial>
-                <origin xyz="${link_length* 0.5 - 0.0576} 0.0 0.0258" rpy="0 0 0"/>
-                <mass value="0.616"/>
+                <origin xyz="${link_length* link_inertial_pos - 0.0576} 0.0 0.0258" rpy="0 0 0"/>
+                <mass value="${0.616-0.3*vibrate}"/>
                 <inertia
                     ixx="0.002" iyy="0.0161" izz="0.016992"
@@ -83,6 +89,6 @@
             <xacro:unless value="${tilt_mode == 1}">
               <inertial>
-                <origin xyz="${link_length * 0.5 -0.058} 0.0 0.0188" rpy="0 0 0"/>
-                <mass value="0.590"/> <!-- +DCDC -->
+                <origin xyz="${link_length * link_inertial_pos -0.058} 0.0 0.0188" rpy="0 0 0"/>
+                <mass value="${0.590-0.3*vibrate}"/> <!-- +DCDC -->
                 <inertia
                     ixx="0.00179" iyy="0.01581" izz="0.01692"
@@ -97,6 +103,6 @@
               <xacro:if value="${tilt_mode == 1}">
                 <inertial>
-                  <origin xyz="${link_length* 0.5 - 0.0005} 0.0 0.0204" rpy="0 0 0"/>
-                  <mass value="0.58312"/>
+                  <origin xyz="${link_length* link_inertial_pos - 0.0005} 0.0 0.0204" rpy="0 0 0"/>
+                  <mass value="${0.58312-0.3*vibrate}"/>
                   <inertia
                       ixx="0.002" iyy="0.01752" izz="0.018447"
@@ -106,6 +112,6 @@
               <xacro:unless value="${tilt_mode == 1}">
                 <inertial>
-                  <origin xyz="${link_length * 0.5} 0.0 0.01287" rpy="0 0 0"/>
-                  <mass value="0.55744"/>
+                  <origin xyz="${link_length * link_inertial_pos} 0.0 0.01287" rpy="0 0 0"/>
+                  <mass value="${0.55744-0.3*vibrate}"/>
                   <inertia
                       ixx="0.00171" iyy="0.01727" izz="0.01844"
@@ -119,6 +125,6 @@
               <xacro:if value="${tilt_mode == 1}">
                 <inertial>
-                  <origin xyz="${link_length* 0.5 - 0.03} 0.0 0.025" rpy="0 0 0"/>
-                  <mass value="0.66183"/>
+                  <origin xyz="${link_length* link_inertial_pos - 0.03} 0.0 0.025" rpy="0 0 0"/>
+                  <mass value="${0.66183-0.3*vibrate}"/>
                   <inertia
                       ixx="0.002" iyy="0.021851" izz="0.022718"
@@ -128,6 +134,6 @@
               <xacro:unless value="${tilt_mode == 1}">
                 <inertial>
-                  <origin xyz="${link_length * 0.5 - 0.0317} 0.0 0.01836" rpy="0 0 0"/>
-                  <mass value="0.63453"/>
+                  <origin xyz="${link_length * link_inertial_pos - 0.0317} 0.0 0.01836" rpy="0 0 0"/>
+                  <mass value="${0.63453-0.3*vibrate}"/>
                   <inertia
                       ixx="0.00182" iyy="0.02232" izz="0.02254"
@@ -241,10 +247,9 @@
         <link name="torsion_dummy${self}">
           <inertial>
-            <origin xyz="0 0 0" rpy="0 0 0"/>
-            <mass value="0.001"/>
+            <origin xyz="${link_length*0.25} 0 0.012" rpy="0 0 0"/>
+            <mass value="0.3"/>
             <inertia
-                ixx="0.0001" ixy="0.0" ixz="0.0"
-                iyy="0.0001" iyz="0.0"
-                izz="0.0002"/>
+                ixx="0.001828" iyy="0.021127" izz="0.022388"
+                ixy="0.000021" ixz="0.000260" iyz="0.000000"/>
           </inertial>
         </link>
@@ -253,26 +258,8 @@
           <parent link="link${self}"/>
           <child link="torsion_dummy${self}"/>
-          <origin rpy="0 0 0" xyz="${link_length} 0 0"/>
+          <origin rpy="0 0 0" xyz="${link_length/2} 0 0"/>
           <axis xyz="1 0 0"/>
-          <dynamics damping="0.7" friction="0.00"/>
+          <dynamics damping="1.0" friction="0.00"/>
         </joint>
-        <!-- <link name="torsion_dummy${self}_l"> -->
-        <!--   <inertial> -->
-        <!--     <origin xyz="0 0 0" rpy="0 0 0"/> -->
-        <!--     <mass value="0.001"/> -->
-        <!--     <inertia -->
-        <!--         ixx="0.0001" ixy="0.0" ixz="0.0" -->
-        <!--         iyy="0.0001" iyz="0.0" -->
-        <!--         izz="0.0002"/> -->
-        <!--   </inertial> -->
-        <!-- </link> -->
-        <!-- <joint name="torsion${self}_l" type="revolute"> -->
-        <!--   <limit effort="10000.0" lower="${-pi/6}" upper="${pi/6}" velocity="1"/> -->
-        <!--   <parent link="torsion_dummy${self}_l"/> -->
-        <!--   <child link="link${self+1}"/> -->
-        <!--   <origin rpy="0 0 0" xyz="0 0 0"/> -->
-        <!--   <axis xyz="1 0 0"/> -->
-        <!--   <dynamics damping="0.9" friction="0.05"/> -->
-        <!-- </joint> -->
       </xacro:if>
       <joint name="joint${self}" type="revolute">
@@ -286,6 +273,5 @@
           <parent link="torsion_dummy${self}"/>
           <child link="link${self+1}"/>
-          <!-- <child link="torsion_dummy${self}_l"/> -->
-          <origin rpy="0 0 0" xyz="0 0 0"/>
+          <origin rpy="0 0 0" xyz="${link_length*0.5} 0 0"/>
         </xacro:if>
         <axis xyz="0 0 1"/>

Commit message: refactored null space gain shift

File: robots/hydrus/robots/oct/oct_vibration_mode_202010/robot.gazebo.xacro (robot description, xacro)
@@ -12,38 +12,39 @@
   <xacro:gazebo_spinal robot_name="$(arg robot_name)" />
   <xacro:if value="$(arg sim)">
+    <xacro:property name="kx" value="60" />
     <gazebo>
       <!-- joint torsional spring plugin -->
       <plugin name="torsion1_torsional_spring" filename="libjoint_torsional_spring_plugin.so">
-        <kx>60</kx>
+        <kx>${kx}</kx>
         <set_point>0</set_point>
         <joint>torsion1</joint>
       </plugin>
       <plugin name="torsion2_torsional_spring" filename="libjoint_torsional_spring_plugin.so">
-        <kx>60</kx>
+        <kx>${kx}</kx>
         <set_point>0</set_point>
         <joint>torsion2</joint>
       </plugin>
       <plugin name="torsion3_torsional_spring" filename="libjoint_torsional_spring_plugin.so">
-        <kx>60</kx>
+        <kx>${kx}</kx>
         <set_point>0</set_point>
         <joint>torsion3</joint>
       </plugin>
       <plugin name="torsion4_torsional_spring" filename="libjoint_torsional_spring_plugin.so">
-        <kx>60</kx>
+        <kx>${kx}</kx>
         <set_point>0</set_point>
         <joint>torsion4</joint>
       </plugin>
       <plugin name="torsion5_torsional_spring" filename="libjoint_torsional_spring_plugin.so">
-        <kx>60</kx>
+        <kx>${kx}</kx>
         <set_point>0</set_point>
         <joint>torsion5</joint>
       </plugin>
       <plugin name="torsion6_torsional_spring" filename="libjoint_torsional_spring_plugin.so">
-        <kx>60</kx>
+        <kx>${kx}</kx>
         <set_point>0</set_point>
         <joint>torsion6</joint>
       </plugin>
       <plugin name="torsion7_torsional_spring" filename="libjoint_torsional_spring_plugin.so">
-        <kx>60</kx>
+        <kx>${kx}</kx>
         <set_point>0</set_point>
         <joint>torsion7</joint>
