Commit message: modified model

File: robots/hydrus/robots/oct/oct_vibration_shift_202011_task3/robot.urdf.xacro (robot description, xacro)
@@ -189,7 +189,21 @@
   </xacro:extra_module>
   <!-- end: neuron imus -->
+  <!-- 2.3 downwards rs-t265 (VIO) -->
+  <xacro:extra_module name = "realsense1_pose_frame" parent = "link4" visible = "1"
+    model_url = "package://mbzirc2020_common/urdf/mesh/modules/sensor/downward_realsense_unit.STL">
+    <origin xyz="${link_length/2 + 0.127} 0.0 -0.022" rpy="0 ${pi/2} ${pi/2}"/>
+    <inertial>
+      <mass value = "0.065" /> <!-- sensor + usb-cable -->
+      <origin xyz="-0.009 -0.01 0" rpy="0 0 0"/>
+      <inertia
+        ixx="0.0" ixy="0.0" ixz="0.0"
+        iyy="0.0" iyz="0.0"
+        izz="0.0"/>
+    </inertial>
+  </xacro:extra_module>
+  <!-- end: rs-t265 -->
   <!-- 2. FLIR -->
-  <xacro:extra_module name = "lepton_camera" parent = "link4" visible = "0"  >
-    <origin xyz="${link_length / 2 + 0.24455} 0.05545 -0.015" rpy="0 ${pi/2} ${3 * pi/4}"/>
+  <xacro:extra_module name = "lepton_camera" parent = "link5" visible = "0"  >
+    <origin xyz="0.12 0.0 -0.015" rpy="0 ${pi/2} ${0 * pi/4}"/>
     <inertial>
       <mass value = "0.02" />
