Commit message: modified vibration model according to experiment

File: robots/hydrus/robots/oct/oct_vibration_shift_202011/robot.gazebo.xacro (robot description, xacro)
@@ -11,5 +11,5 @@
   <xacro:gazebo_spinal robot_name="$(arg robot_name)" />
   <xacro:if value="$(arg sim)">
-    <xacro:property name="kx" value="60" />
+    <xacro:property name="kx" value="100" />
     <gazebo>
       <!-- joint torsional spring plugin -->
